Commit message: refine the urdf model

File: rrcar_description/urdf/base.urdf.xacro (robot description, xacro)
@@ -4,8 +4,8 @@
 	<xacro:property name="wheel_width" value="0.05" />
 	<xacro:property name="wheel_mass" value="0.3" />
-	<xacro:property name="body_radius" value="0.15" />
-	<xacro:property name="body_height" value="0.049" />
+	<xacro:property name="body_height" value="0.046" />
 	<xacro:property name="body_mass" value="3" />
 	<xacro:property name="track_width" value="0.22" />
+	<xacro:property name="vehicle_height" value="0.004" />
 	<xacro:macro name="wheel_visual">
 		<visual>
@@ -41,11 +41,10 @@
 		<parent link="base_footprint" />
 		<child link="base_link" />
-		<origin xyz="0 0 ${body_height / 2 + 0.001}" rpy="0 0 0" />
+		<origin xyz="0 0 ${vehicle_height}" rpy="0 0 0" />
 	</joint>
 	<link name="base_link">
 		<visual>
-			<origin xyz="0 0 -${body_height / 2}" rpy="${M_PI / 2} 0 ${M_PI / 2}" />
+			<origin xyz="0 0 0" rpy="${M_PI / 2} 0 ${M_PI / 2}" />
 			<geometry>
-				<!-- cylinder radius="${body_radius}" length="${body_height}" / -->
 				<mesh filename="package://rrcar_description/meshes/base_link.stl" />
 			</geometry>
@@ -53,7 +52,6 @@
 		</visual>
 		<collision>
-			<origin xyz="0 0 -${body_height / 2}" rpy="${M_PI / 2} 0 ${M_PI / 2}" />
+			<origin xyz="0 0 0" rpy="${M_PI / 2} 0 ${M_PI / 2}" />
 			<geometry>
-				<!-- cylinder radius="${body_radius}" length="${body_height}" / -->
 				<mesh filename="package://rrcar_description/meshes/base_link.stl" />
 			</geometry>
@@ -65,5 +63,5 @@
 		<parent link="base_link" />
 		<child link="wheel_left" />
-		<origin xyz="0 ${track_width / 2} ${body_height / 2 - 0.003}" rpy="0 0 0" />
+		<origin xyz="0 ${track_width / 2} ${wheel_radius - vehicle_height}" rpy="0 0 0" />
 		<axis xyz="0 1 0" />
 		<limit effort="8" velocity="30.0" />
@@ -79,5 +77,5 @@
 		<parent link="base_link" />
 		<child link="wheel_right" />
-		<origin xyz="0 -${track_width / 2} ${body_height / 2 - 0.003}" rpy="0 0 0" />
+		<origin xyz="0 -${track_width / 2} ${wheel_radius - vehicle_height}" rpy="0 0 0" />
 		<axis xyz="0 -1 0" />
 		<limit effort="8" velocity="30.0" />
@@ -93,5 +91,5 @@
 	<joint name="camera_joint" type="fixed">
 		<axis xyz="0 1 0" />
-		<origin xyz="0.1 0 ${body_height / 2 + 0.05 / 2 - 0.002}" rpy="0 0 0"/>
+		<origin xyz="0.14 0 0.04" rpy="0 0 0"/>
 		<parent link="base_link"/>
 		<child link="camera_link"/>
@@ -101,5 +99,5 @@
 			<origin xyz="0 0 0" rpy="0 0 0"/>
 			<geometry>
-				<box size="0.05 0.05 0.05"/>
+				<box size="0.02 0.02 0.01"/>
 			</geometry>
 		</collision>
@@ -107,17 +105,17 @@
 			<origin xyz="0 0 0" rpy="0 0 0"/>
 			<geometry>
-				<box size="0.05 0.05 0.05"/>
+				<box size="0.02 0.02 0.01"/>
 			</geometry>
-			<xacro:material_light_gray />
+			<xacro:material_red />
 		</visual>
 		<inertial>
-			<mass value="1e-5" />
+			<mass value="1e-4" />
 			<origin xyz="0 0 0" rpy="0 0 0"/>
-			<inertia ixx="1e-6" ixy="0" ixz="0" iyy="1e-6" iyz="0" izz="1e-6" />
+			<inertia ixx="1e-5" ixy="0" ixz="0" iyy="1e-5" iyz="0" izz="1e-5" />
 		</inertial>
 	</link>
 	<joint name="hokuyo_joint" type="fixed">
 		<axis xyz="0 0 1" />
-		<origin xyz="0.1 0 ${body_height / 2 + 0.05 / 2 + 0.05 - 0.002}" rpy="0 0 0"/>
+		<origin xyz="0.13 0 ${body_height}" rpy="0 0 0"/>
 		<parent link="base_link"/>
 		<child link="hokuyo_link"/>
@@ -125,20 +123,20 @@
 	<link name="hokuyo_link">
 		<collision>
-			<origin xyz="0 0 0" rpy="0 0 0"/>
+			<origin xyz="0 0 ${0.029 / 2}" rpy="0 0 0"/>
 			<geometry>
-				<box size="0.05 0.05 0.05"/>
+				<cylinder radius="0.021" length="0.029"/>
 			</geometry>
 		</collision>
 		<visual>
-			<origin xyz="0 0 0" rpy="0 0 0"/>
+			<origin xyz="0 0 ${0.029 / 2}" rpy="0 0 0"/>
 			<geometry>
-				<box size="0.05 0.05 0.05"/>
+				<cylinder radius="0.021" length="0.029"/>
 			</geometry>
 			<xacro:material_black />
 		</visual>
 		<inertial>
-			<mass value="1e-5" />
+			<mass value="0.16" />
 			<origin xyz="0 0 0" rpy="0 0 0"/>
-			<inertia ixx="1e-6" ixy="0" ixz="0" iyy="1e-6" iyz="0" izz="1e-6" />
+			<inertia ixx="0.016" ixy="0" ixz="0" iyy="0.016" iyz="0" izz="0.016" />
 		</inertial>
 	</link>
