Commit message: [cube_description] modified parameters of the robot

File: rrcar_description/urdf/common_properties.urdf.xacro (robot description, xacro)
@@ -10,6 +10,6 @@
 			<origin xyz="${origin_xyz}" />
 			<inertia ixx="1.0" ixy="0.0" ixz="0.0"
-													iyy="1.0" iyz="0.0"
-																		izz="1.0" />
+				 iyx="0.0" iyy="1.0" iyz="0.0"
+				 izx="0.0" izy="0.0" izz="1.0" />
 		</inertial>
 	</xacro:macro>

File: rrcar_description/urdf/rrcar.urdf.xacro (robot description, xacro)
@@ -5,5 +5,5 @@
 	<xacro:property name="wheel_mass" value="0.3" />
 	<xacro:property name="body_height" value="0.046" />
-	<xacro:property name="body_mass" value="3" />
+	<xacro:property name="body_mass" value="8" />
 	<xacro:property name="track_width" value="0.22" />
 	<xacro:property name="vehicle_height" value="0.004" />
