Commit message: [rrcar_control, rrcar_description] use diff_drive_controller

File: rrcar_description/urdf/rrcar.urdf.xacro (robot description, xacro)
@@ -65,5 +65,5 @@
 		<origin xyz="0 ${track_width / 2} ${wheel_radius - vehicle_height}" rpy="0 0 0" />
 		<axis xyz="0 1 0" />
-		<limit effort="8" velocity="30.0" />
+		<limit effort="2" velocity="10.0" />
 		<dynamics damping="0.3" friction="0.2" />
 	</joint>
@@ -78,6 +78,6 @@
 		<child link="wheel_right" />
 		<origin xyz="0 -${track_width / 2} ${wheel_radius - vehicle_height}" rpy="0 0 0" />
-		<axis xyz="0 -1 0" />
-		<limit effort="8" velocity="30.0" />
+		<axis xyz="0 1 0" />
+		<limit effort="2" velocity="10.0" />
 		<dynamics damping="0.3" friction="0.2" />
 	</joint>

Commit message: [rrcar_description] add an IMU

File: rrcar_description/urdf/rrcar.urdf.xacro (robot description, xacro)
@@ -141,4 +141,11 @@
 		</inertial>
 	</link>
+	<joint name="imu_joint" type="fixed">
+		<axis xyz="0 0 1" />
+		<origin xyz="0 0 0" rpy="0 0 0" />
+		<parent link="base_link" />
+		<child link="imu_link" />
+	</joint>
+	<link name="imu_link" />
   <xacro:include filename="$(find rrcar_description)/urdf/rrcar.gazebo" />
 </robot>
